File: usb_hub.kicad_pcb (KiCad board)
At the start: 2 copper layers, 120 x 65 mm, 21 parts, among them J1 CONN_01X02_MALE-B2B, J10 USB_A, J11 USB_A, J12 USB_A, J13 USB_A, J14 USB_A, J15 USB_A, J16 USB_A, J17 USB_A, J18 CONN_COAXIAL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

Commit message: corrected pcb outline
Parts:
- removed J1, J2: CONN_01X02_MALE-B2B, Connectors_Molex:Molex_MiniFit-JR-5556-02A_2x01x4.20mm_Straight
- removed J10, J11, J12, J13, J14, J15, J16, J17, J6, J7: USB_A, Connectors:USB_A
- removed J18, J19, J20, J21: CONN_COAXIAL, Connectors:BARREL_JACK
- removed J3: DIL24, Connectors_Molex:Molex_MiniFit-JR-5556-24A_2x12x4.20mm_Straight
- removed J4, J5, J8, J9: CONN_01X02_MALE, Connectors_JST:JST_XH_B02B-XH-A_02x2.50mm_Straight
- added REF** (x2): ATX_Wire_On_Board, Connectors:IDC_Header_Straight_20pins, F.Cu at (0.00, 0.00)
Other:
- board outline removed
- board text removed: "15 June 2017"
- board text removed: "A"
- board text removed: "Raspberry Pi 3 SMPS powered USB Hub"
