File: usb_hub.sch (KiCad schematic (older format))
At the start: 20 parts, among them J1 USB_A, J10 USB_A, J11 CONN_01X04_MALE, J12 DIL24, J13 CONN_01X02_MALE, J14 CONN_01X02_MALE, J15 CONN_01X02_MALE, J16 CONN_01X02_MALE, J17 CONN_COAXIAL, J18 CONN_COAXIAL, J19 CONN_COAXIAL, J2 USB_A, J20 CONN_COAXIAL, J3 USB_A, J4 USB_A, J5 USB_A, J6 USB_A, J7 USB_A, J8 USB_A, J9 USB_A

Commit message: A.1
Parts:
- removed J11: CONN_01X04_MALE, symbol CONN_01X04_MALE
- added J1, J2: CONN_01X02_MALE-B2B, Connectors_Molex:Molex_MiniFit-JR-5556-02A_2x01x4.20mm_Straight, symbol CONN_01X02_MALE
- J4: renamed from J13; footprint (none) -> Connectors_JST:JST_XH_B02B-XH-A_02x2.50mm_Straight
- J5: renamed from J14; footprint (none) -> Connectors_JST:JST_XH_B02B-XH-A_02x2.50mm_Straight
- J8: renamed from J15; footprint (none) -> Connectors_JST:JST_XH_B02B-XH-A_02x2.50mm_Straight
- J9: renamed from J16; footprint (none) -> Connectors_JST:JST_XH_B02B-XH-A_02x2.50mm_Straight
- renumbered J3 to J10, J4 to J11, J5 to J12, J6 to J13, J7 to J14, J8 to J15, J9 to J16, J10 to J17, J17 to J18, J18 to J19, J19 to J20, J20 to J21, J12 to J3, J1 to J6, J2 to J7
Connections:
- net +12V: now also J1.1
- net +3V3: now also J3.13 (P13); no longer J3.24 (P24)
- net +5V: now also J3.21 (P21), J3.22 (P22), J3.23 (P23), J2.2; no longer J3.14 (P14), J3.15 (P15), J3.16 (P16)
- net +5VSB: now also J3.9 (P9); no longer J3.8 (P8)
- net -12VA: now also J3.14 (P14); no longer J3.23 (P23)
- net GND: now also J3.15 (P15), J3.16 (P16), J3.17 (P17), J3.24 (P24), J1.2, J2.1; no longer J3.13 (P13), J3.20 (P20), J3.21 (P21), J3.22 (P22)
- net POWER_OK: now also J3.8 (P8); no longer J3.9 (P9)

Commit message: corrected pcb outline
Parts:
- J3: footprint Connectors_Molex:Molex_MiniFit-JR-5556-24A_2x12x4.20mm_Straight -> Custom_Connectors:ATX_Wire_On_Board
Changed lines of the file:
@@
 F 0 "J3" H 2550 2100 50  0000 C CNN
 F 1 "DIL24" H 2550 1900 50  0000 C CNN
-F 2 "Connectors_Molex:Molex_MiniFit-JR-5556-24A_2x12x4.20mm_Straight" H 2550 2000 50  0001 C CNN
+F 2 "Custom_Connectors:ATX_Wire_On_Board" H 2550 2000 50  0001 C CNN
 F 3 "" H 2550 2000 50  0001 C CNN
 	1    2550 2000
