File: usb_hub.sch (KiCad schematic (older format))
At the start: 21 parts, among them J1 CONN_01X02_MALE-B2B, J10 USB_A, J11 USB_A, J12 USB_A, J13 USB_A, J14 USB_A, J15 USB_A, J16 USB_A, J17 USB_A, J18 CONN_COAXIAL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

Commit message: Rev A complete
Parts:
- removed J13, J6: USB_A, Connect:USB_A, symbol USB_A
- removed J18, J21: CONN_COAXIAL, Connectors:BARREL_JACK, symbol CONN_COAXIAL
- J3: footprint Connectors_Molex:Molex_MiniFit-JR-5556-24A_2x12x4.20mm_Straight -> Custom_Connectors:ATX_Wire_On_Board
Connections:
- net +5V: now also J2.1; no longer J2.2
- net GND: now also J2.2; no longer J2.1
- no-connect marks 31 -> 25
Other:
- moved on the sheet: J11, J12, J14, J15, J16, J17, J7
